Commit message: 20211203

File: pcl_processor/urdf/realsense_435_demo_robot.urdf.xacro (robot description, xacro)
@@ -7,5 +7,5 @@
   <!-- Realsense Camera Joint Position -->
   <xacro:sensor_d435 parent="world" use_nominal_extrinsics="true">
-    <origin xyz="0.0 0.00 0.7" rpy="0 1.57 0"/>
+    <origin xyz="0.0 0.00 0.5" rpy="0 1.57 0"/>
   </xacro:sensor_d435>
 </robot>
